File: hardware/pcb/mothership-nrf52840-xiao-rev1-matt/mothership.kicad_sch (KiCad schematic)
At the start: 42 parts, among them J1 HRO TYPE-C-31-M-12, J10 CONN_BATT, J11 Screw_Terminal_ADB_VCC, J2 USB_EXT_FFC_CABLE, J3 Screw_Terminal_ADB_SHIELD, J4 CONN_MATRIX_BOT_L, J5 CONN_MATRIX_BOT_R, J6 CONN_MATRIX_TOP_R, J7 CONN_MATRIX_TOP_L, J8 SPI, J9 EC11, Q1 AO3401A, Q2 FDC6305N, SW1 SW_SPDT_321, SW2 SW_SPST, U1 NCP361SN, U2 XIAO_nRF52840, U3 MCP23017x-x-SS, U4 MCP23017x-x-SS, U5 DT1452-02SO, U6 HY2115-LB9D

Commit message: sch: fix typo for batt ic series in R value recommendation
Other:
- note added: "Avoid Kelvin pick-up Should originate from the Resistor pad"
- note added: "R1: BPROT VDD FEED HY2115/HY2113: 100R S-8261A: 470R S-8240Â: 330R R2: BPROT NEG-SENSE LIMIT 2K00 DEFAULT S-8240A: 470R R3: BPROT_SHUNT/BYPASS HY2115: 100mR 1% LOW-TCR; CLASSIC: LOW-R 0R JUMPER R4: CS_LINK HY2115: 0R; CLASSIC: DNP"
- note removed: "R1: BPROT VDD FEED HY2115/HY2113: 100R S-8261A: 470R S-8240D: 330R R2: BPROT NEG-SENSE LIMIT 2K00 DEFAULT S-8240D: 470R R3: BPROT_SHUNT/BYPASS HY2115: 100mR 1% LOW-TCR; CLASSIC: LOW-R 0R JUMPER R4: CS_LINK HY2115: 0R; CLASSIC: DNP"
- moved on the sheet: R10
Changed lines of the file:
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@@
 		)
 	)
-	(text "R1: BPROT VDD FEED\n    HY2115/HY2113: 100R \n    S-8261A: 470R\n    S-8240D: 330R\n\nR2: BPROT NEG-SENSE LIMIT\n    2K00 DEFAULT\n    S-8240D: 470R\n\nR3: BPROT_SHUNT/BYPASS\n    HY2115: 100mR 1% LOW-TCR;\n    CLASSIC: LOW-R 0R JUMPER\n\nR4: CS_LINK\n    HY2115: 0R;\n    CLASSIC: DNP"
+	(text "R1: BPROT VDD FEED\n    HY2115/HY2113: 100R \n    S-8261A: 470R\n    S-8240Â: 330R\n\nR2: BPROT NEG-SENSE LIMIT\n    2K00 DEFAULT\n    S-8240A: 470R\n\nR3: BPROT_SHUNT/BYPASS\n    HY2115: 100mR 1% LOW-TCR;\n    CLASSIC: LOW-R 0R JUMPER\n\nR4: CS_LINK\n    HY2115: 0R;\n    CLASSIC: DNP"
 		(exclude_from_sim no)
 		(at 318.008 121.158 0)
@@
 		)
 	)
+	(text "Avoid Kelvin pick-up\nShould originate from \nthe Resistor pad"
+		(exclude_from_sim no)
+		(at 241.808 172.72 0)
+		(effects
+			(font
+				(size 0.889 0.889)
+			)
+			(justify left)
+		)
+	)
 	(text "Pins to Matrix\n--------------"
 		(exclude_from_sim no)
@@
 	)
 	(junction
-		(at 246.38 151.13)
-		(diameter 0)
-		(color 0 0 0 0)
-	)
-	(junction
 		(at 105.41 38.1)
 		(diameter 0)
@@
 	(wire
 		(pts
-			(xy 246.38 162.56) (xy 250.19 162.56)
-		)
-		(stroke
-			(width 0)
-			(type default)
-		)
-	)
-	(wire
-		(pts
 			(xy 233.68 46.99) (xy 232.41 46.99)
 		)
@@
 	(wire
 		(pts
+			(xy 248.92 153.67) (xy 261.62 153.67)
+		)
+		(stroke
+			(width 0)
+			(type default)
+		)
+	)
+	(wire
+		(pts
 			(xy 64.77 217.17) (xy 62.23 217.17)
 		)
@@
 	(wire
 		(pts
+			(xy 261.62 153.67) (xy 261.62 151.13)
+		)
+		(stroke
+			(width 0)
+			(type default)
+		)
+	)
+	(wire
+		(pts
 			(xy 62.23 250.19) (xy 62.23 251.46)
 		)
@@
 	(wire
 		(pts
-			(xy 243.84 151.13) (xy 246.38 151.13)
+			(xy 243.84 151.13) (xy 261.62 151.13)
 		)
 		(stroke
@@
 	(wire
 		(pts
-			(xy 214.63 20.32) (xy 214.63 19.05)
+			(xy 248.92 162.56) (xy 248.92 153.67)
 		)
 		(stroke
@@
 	(wire
 		(pts
-			(xy 243.84 146.05) (xy 248.92 146.05)
+			(xy 214.63 20.32) (xy 214.63 19.05)
 		)
 		(stroke
@@
 	(wire
 		(pts
-			(xy 81.28 45.72) (xy 88.9 45.72)
+			(xy 243.84 146.05) (xy 248.92 146.05)
 		)
 		(stroke
@@
 	(wire
 		(pts
-			(xy 40.64 119.38) (xy 40.64 127)
+			(xy 81.28 45.72) (xy 88.9 45.72)
 		)
 		(stroke
@@
 	(wire
 		(pts
-			(xy 275.59 180.34) (xy 275.59 182.88)
+			(xy 40.64 119.38) (xy 40.64 127)
 		)
 		(stroke
@@
 	(wire
 		(pts
-			(xy 59.69 224.79) (xy 59.69 231.14)
+			(xy 275.59 180.34) (xy 275.59 182.88)
 		)
 		(stroke
@@
 	(wire
 		(pts
-			(xy 255.27 162.56) (xy 257.81 162.56)
+			(xy 59.69 224.79) (xy 59.69 231.14)
 		)
 		(stroke
@@
 	(wire
 		(pts
-			(xy 189.23 143.51) (xy 189.23 146.05)
+			(xy 248.92 162.56) (xy 252.73 162.56)
 		)
 		(stroke
@@
 	(wire
 		(pts
-			(xy 246.38 151.13) (xy 261.62 151.13)
+			(xy 189.23 143.51) (xy 189.23 146.05)
 		)
 		(stroke
@@
 	(wire
 		(pts
-			(xy 246.38 151.13) (xy 246.38 162.56)
-		)
-		(stroke
-			(width 0)
-			(type default)
-		)
-	)
-	(wire
-		(pts
 			(xy 137.16 57.15) (xy 148.59 57.15)
 		)
@@
 	(symbol
 		(lib_id "A9M0330:R_Small")
-		(at 252.73 162.56 90)
+		(at 255.27 162.56 90)
 		(mirror x)
 		(unit 1)
@@
 		(dnp no)
 		(property "Reference" "R10"
-			(at 254.254 157.988 90)
+			(at 256.794 157.988 90)
 			(show_name no)
 			(do_not_autoplace no)
@@
 		)
 		(property "Value" "BPROT_SHUNT/BYPASS"
-			(at 252.73 160.02 90)
+			(at 255.27 160.02 90)
 			(show_name no)
 			(do_not_autoplace no)
@@
 		)
 		(property "Footprint" "A9M0330:Resistor_SMD__R_0603_1608Metric_Pad0.98x0.95mm_HandSolder"
-			(at 252.73 162.56 0)
+			(at 255.27 162.56 0)
 			(hide yes)
 			(show_name no)
@@
 		)
 		(property "Datasheet" ""
-			(at 252.73 162.56 0)
+			(at 255.27 162.56 0)
 			(hide yes)
 			(show_name no)
@@
 		)
 		(property "Description" "Resistor, small symbol"
-			(at 252.73 162.56 0)
+			(at 255.27 162.56 0)
 			(hide yes)
 			(show_name no)
